Commit message: MUIN First commit

File: scout/scout_description/urdf/custard.xacro (robot description, xacro)
@@ -66,4 +66,7 @@
         <child link="base_link"/>
     </joint> -->
+    <gazebo reference="livox_frame">
+        <material>Gazebo/LightBlueLaser</material>
+    </gazebo>
     <!-- Scout wheel macros -->
     <!-- wheel labeled from 0 to 3, conter-clockwise, starting from front right wheel -->
@@ -93,4 +96,9 @@
         <origin xyz="${-wheelbase/2} ${-track/2} ${wheel_vertical_offset+0.001}" rpy="1.57 0 0" />
     </xacro:scout_mini_wheel_4>
+    <!-- Lidar Sensor -->
+    <xacro:include filename="$(find ros2_livox_simulation)/urdf/mid360.xacro" />
+    <xacro:mid360 name="livox_frame" parent="base_link" topic="/livox/lidar">
+        <origin xyz="0 0 0.45" rpy="0 0 0"/>
+    </xacro:mid360>
     <!-- Additional definitions -->
     <xacro:include filename="$(arg urdf_extras)" />

File: scout/scout_description/urdf/scout_mini_wheel_1.xacro (robot description, xacro)
@@ -36,5 +36,5 @@
                 <origin xyz="0 0 0" rpy="0 0 0" />
                 <geometry>
-                    <mesh filename="package://scout_description/meshes/wheel.dae" />
+                    <mesh filename="file://$(find scout_description)/meshes/wheel.dae" />
                 </geometry>
             </visual>-->
@@ -48,5 +48,5 @@
                 <origin xyz="0 0 0" rpy="0 0 0" />
                 <geometry>
-                    <mesh filename="package://scout_description/meshes/wheel.dae" />
+                    <mesh filename="file://$(find scout_description)/meshes/wheel.dae" />
                 </geometry>
             </visual>
@@ -57,5 +57,5 @@
               <geometry>
                 <mesh
-                  filename="package://scout_description/meshes/wheel.dae" />
+                  filename="file://$(find scout_description)/meshes/wheel.dae" />
               </geometry>
             </collision>
@@ -68,5 +68,5 @@
             <child link="${wheel_prefix}_wheel_link"/>
             <xacro:insert_block name="joint_pose"/>
-            <axis xyz="0 0 -1" rpy="0 0 0" />
+            <axis xyz="0 0 1" rpy="0 0 0" />
         </joint>
     </xacro:macro>

File: scout/scout_description/urdf/scout_mini_wheel_2.xacro (robot description, xacro)
@@ -36,5 +36,5 @@
                 <origin xyz="0 0 0" rpy="0 0 0" />
                 <geometry>
-                    <mesh filename="package://scout_description/meshes/wheel.dae" />
+                    <mesh filename="file://$(find scout_description)/meshes/wheel.dae" />
                 </geometry>
             </visual>-->
@@ -48,5 +48,5 @@
                 <origin xyz="0 0 0" rpy="0 0 0" />
                 <geometry>
-                    <mesh filename="package://scout_description/meshes/wheel.dae" />
+                    <mesh filename="file://$(find scout_description)/meshes/wheel.dae" />
                 </geometry>
             </visual>
@@ -57,5 +57,5 @@
               <geometry>
                 <mesh
-                  filename="package://scout_description/meshes/wheel.dae" />
+                  filename="file://$(find scout_description)/meshes/wheel.dae" />
               </geometry>
             </collision>
@@ -68,5 +68,5 @@
             <child link="${wheel_prefix}_wheel_link"/>
             <xacro:insert_block name="joint_pose"/>
-            <axis xyz="0 0 -1" rpy="0 0 0" />
+            <axis xyz="0 0 1" rpy="0 0 0" />
         </joint>
     </xacro:macro>

File: scout/scout_description/urdf/scout_mini_wheel_3.xacro (robot description, xacro)
@@ -36,5 +36,5 @@
                 <origin xyz="0 0 0" rpy="0 0 0" />
                 <geometry>
-                    <mesh filename="package://scout_description/meshes/wheel.dae" />
+                    <mesh filename="file://$(find scout_description)/meshes/wheel.dae" />
                 </geometry>
             </visual>-->
@@ -48,5 +48,5 @@
                 <origin xyz="0 0 0" rpy="0 0 0" />
                 <geometry>
-                    <mesh filename="package://scout_description/meshes/wheel.dae" />
+                    <mesh filename="file://$(find scout_description)/meshes/wheel.dae" />
                 </geometry>
             </visual>
@@ -57,5 +57,5 @@
               <geometry>
                 <mesh
-                  filename="package://scout_description/meshes/wheel.dae" />
+                  filename="file://$(find scout_description)/meshes/wheel.dae" />
               </geometry>
             </collision>

File: scout/scout_description/urdf/scout_mini_wheel_4.xacro (robot description, xacro)
@@ -36,5 +36,5 @@
             <origin xyz="0 0 0" rpy="0 0 0" />
             <geometry>
-                <mesh filename="package://scout_description/meshes/wheel.dae" />
+                <mesh filename="file://$(find scout_description)/meshes/wheel.dae" />
             </geometry>
         </visual>-->
@@ -48,5 +48,5 @@
             <origin xyz="0 0 0" rpy="0 0 0" />
             <geometry>
-                <mesh filename="package://scout_description/meshes/wheel.dae" />
+                <mesh filename="file://$(find scout_description)/meshes/wheel.dae" />
             </geometry>
         </visual>
@@ -57,5 +57,5 @@
               <geometry>
                 <mesh
-                  filename="package://scout_description/meshes/wheel.dae" />
+                  filename="file://$(find scout_description)/meshes/wheel.dae" />
               </geometry>
             </collision>

File: scout/scout_description/urdf/scout_v2.xacro (robot description, xacro)
@@ -22,5 +22,5 @@
             <origin xyz="0 0 0" rpy="0 0 0" />
             <geometry>
-                <mesh filename="package://scout_description/meshes/base_link.dae" />
+                <mesh filename="file://$(find scout_description)/meshes/base_link.dae" />
             </geometry>
         </visual>
@@ -74,10 +74,10 @@
         <origin xyz="${wheelbase/2} ${track/2} ${wheel_vertical_offset}" rpy="0 0 0" />
     </xacro:scout_wheel_type2>
-    <xacro:scout_wheel_type1 wheel_prefix="rear_left">
+    <xacro:scout_wheel_type2 wheel_prefix="rear_left">
         <origin xyz="${-wheelbase/2} ${track/2} ${wheel_vertical_offset}" rpy="0 0 0" />
+    </xacro:scout_wheel_type2>
+    <xacro:scout_wheel_type1 wheel_prefix="rear_right">
+        <origin xyz="${-wheelbase/2} ${-track/2} ${wheel_vertical_offset}" rpy="3.14 0 0" />
     </xacro:scout_wheel_type1>
-    <xacro:scout_wheel_type2 wheel_prefix="rear_right">
-        <origin xyz="${-wheelbase/2} ${-track/2} ${wheel_vertical_offset}" rpy="3.14 0 0" />
-    </xacro:scout_wheel_type2>
     <!-- Additional definitions -->
     <xacro:include filename="$(arg urdf_extras)" />

File: scout/scout_description/urdf/scout_wheel_type1.xacro (robot description, xacro)
@@ -34,5 +34,5 @@
                 <origin xyz="0 0 0" rpy="0 0 0" />
                 <geometry>
-                    <mesh filename="package://scout_description/meshes/wheel_type1.dae" />
+                    <mesh filename="file://$(find scout_description)/meshes/wheel_type1.dae" />
                 </geometry>
             </visual>

File: scout/scout_description/urdf/scout_wheel_type2.xacro (robot description, xacro)
@@ -34,5 +34,5 @@
                 <origin xyz="0 0 0" rpy="0 0 0" />
                 <geometry>
-                    <mesh filename="package://scout_description/meshes/wheel_type1.dae" />
+                    <mesh filename="file://$(find scout_description)/meshes/wheel_type1.dae" />
                 </geometry>
             </visual>
@@ -53,5 +53,5 @@
             <child link="${wheel_prefix}_wheel_link"/>
             <xacro:insert_block name="joint_pose"/>
-            <axis xyz="0 -1 0" rpy="0 0 0" />
+            <axis xyz="0 1 0" rpy="0 0 0" />
             <dynamics damping="0.0" friction="20"/>
         </joint>
